File: AnalogDrum_Modules/AnalogDrum_FM/AnalogDrum_FM.sch (KiCad schematic (older format))
At the start: 13 parts, among them J101 Conn_01x05_Male, SW101 SW_SPDT, SW102 SW_SPDT

Commit message: Version 0.1.1
Corrections mineures :
- Vérification des potentiomètres
- Passage des connecteurs de carte e n JST
Parts:
- J101: footprint Connector_PinHeader_2.54mm:PinHeader_1x05_P2.54mm_Horizontal -> Connector_JST:JST_EH_B5B-EH-A_1x05_P2.50mm_Vertical
Changed lines of the file:
@@
 F 0 "J101" H 2008 4681 50  0000 C CNN
 F 1 "Conn_01x05_Male" H 2008 4590 50  0000 C CNN
-F 2 "Connector_PinHeader_2.54mm:PinHeader_1x05_P2.54mm_Horizontal" H 1900 4300 50  0001 C CNN
+F 2 "Connector_JST:JST_EH_B5B-EH-A_1x05_P2.50mm_Vertical" H 1900 4300 50  0001 C CNN
 F 3 "~" H 1900 4300 50  0001 C CNN
 	1    1900 4300
